Commit message: Add essential scripts and update URDF with mimic joint for arm control
- Added all essential ROS 2 and MuJoCo scripts into the `scripts/` folder with a detailed README.
- Included `generate_particle.py`, `gotopose.py`, `grasp.py`, `keyboard_teleop.py`, `rotate_base.py`, and `command_jtc.ipynb` with explanations and features.
- Updated URDF to add mimic joint tags for the arm, enabling coordinated motion of linked joints.
- Verified arm movement using `joint_trajectory_controller`; functionality works but is still under development.
- README now contains a table with hyperlinks to each script/notebook with detailed descriptions.

File: example/hello_robot_stretch_3/stretch.urdf (robot description, URDF)
Before this commit: robot stretch, 37 links, 38 joints
Joints:
- joint joint_arm_l1: mimic (none) -> joint=joint_arm_l0 multiplier=1.0 offset=0.0
- joint joint_arm_l2: mimic (none) -> joint=joint_arm_l0 multiplier=1.0 offset=0.0
- joint joint_arm_l3: mimic (none) -> joint=joint_arm_l0 multiplier=1.0 offset=0.0
